File: Hardware/Adapter/Adapter.kicad_pcb (KiCad board)
At the start: 2 copper layers, 14 parts, among them J1 GameBoy_LinkPort, Q1 BSS13B, Q2 BSS13B, Q3 BSS13B, Q4 BSS13B, U1 Pico

Commit message: More work on adapter
Parts:
- J1, Q1, Q2, Q3, Q4, R1, R2, R3, R4, R5, R6, R7, R8: moved to B.Cu
- moved J1 32.8 mm to (163.9, 82.1), turned to 90 degrees
- moved R8 27.5 mm to (133.6, 90.7), turned to -90 degrees
- moved R6 27.5 mm to (138.4, 90.7), turned to -90 degrees
- moved R5 27.5 mm to (143.3, 90.7), turned to -90 degrees
- moved R7 27.4 mm to (148.1, 90.7), turned to -90 degrees
- moved Q4 21.0 mm to (133.6, 94.0), turned to 90 degrees
- moved Q2 20.9 mm to (138.4, 94.0), turned to 90 degrees
- moved Q1 20.9 mm to (143.3, 94.0), turned to 90 degrees
- moved Q3 20.9 mm to (148.1, 94.0), turned to 90 degrees
- moved R4 14.5 mm to (133.6, 97.3), turned to -90 degrees
- moved R2 14.5 mm to (138.4, 97.3), turned to -90 degrees
- moved R1 14.4 mm to (143.3, 97.3), turned to -90 degrees
- moved R3 14.4 mm to (148.1, 97.3), turned to -90 degrees
- moved U1 1.29 mm to (151.9, 94.0)
Routing:
- net +5V: track 121.8 -> 64.5 mm, vias 1 -> 0
- net Net-(J1-Pad4): track 24.0 -> 39.5 mm, vias 0 -> 1
- net Net-(J1-Pad3): track 46.0 -> 34.3 mm, vias 0 -> 1
- net unconnected-(J1-PadSH): track 0.00 -> 8.40 mm
- net +3V3: track 53.2 -> 45.1 mm, vias 0 -> 4
- net Net-(J1-Pad2): track 31.5 -> 38.7 mm, vias 0 -> 1
- net Net-(J1-Pad5): track 40.8 -> 36.5 mm
- net GND: track 17.5 -> 14.1 mm
- net PSC: track 21.3 -> 17.9 mm
- net PSO: track 23.3 -> 20.8 mm
- net PSI: track 23.4 -> 21.7 mm
- net PSD: track 25.5 -> 26.7 mm
Other:
- board outline added: 52.8 x 32.5 mm
- board text added: "5v"
- board text added: "GND"

Commit message: Not much work at all tbh, trying and failing to import to blender
Parts:
- added G1: LOGO, Gekkio_Connector:SSG Logo, B.Cu at (170.4, 93.7)
Routing:
- net GND: track 14.1 -> 0.00 mm
- net PSI: track 21.7 -> 21.2 mm
- added copper zone on B.Cu, net GND
Other:
- board text added: "Little bit of extra space for wiring"
- board text added: "Oh no! Your Raspberry pi Pico has been stolen! (Totally didn't steal that joke from Stacksmashing)"
- board text added: "TileWorld adapter v.1 Made by: Matthew Collier (Squaresweets) Thanks to: DFranx, Nonchip, Lorenzoone, EchelonPrime, Stacksmashing and maciel310 for making this project possible!"
- board text added: "level shifter thingamabobs"

Commit message: Redid adapter, almost done, but I just wanna code stuff now
Parts:
- removed Q1, Q2, Q3, Q4: BSS13B, Package_TO_SOT_SMD:SOT-23
- removed R1, R2, R3, R4, R5, R6, R7, R8: 10k, Resistor_SMD:R_0402_1005Metric
- moved G1 20.9 mm to (152.1, 103.9)
- moved J1 17.3 mm to (152.7, 95.4)
- moved U1 13.2 mm to (152.1, 107.2)
Connections:
- J1 pad 1: +5V -> unconnected-(J1-Pad1)
- J1 pad 2: Net-(J1-Pad2) -> PSO
- J1 pad 3: Net-(J1-Pad3) -> PSI
- J1 pad 4: Net-(J1-Pad4) -> PSD
- J1 pad 5: Net-(J1-Pad5) -> PSC
- U1 pad 13: GND -> unconnected-(U1-Pad13)
- U1 pad 24: unconnected-(U1-Pad24) -> PSD
- U1 pad 25: unconnected-(U1-Pad25) -> PSO
- U1 pad 26: unconnected-(U1-Pad26) -> PSI
- U1 pad 27: unconnected-(U1-Pad27) -> PSC
Routing:
- net +5V: track 64.5 -> 0.00 mm
- net +3V3: track 45.1 -> 0.00 mm, vias 4 -> 0
- net Net-(J1-Pad4): track 39.5 -> 0.00 mm, vias 1 -> 0
- net Net-(J1-Pad2): track 38.7 -> 0.00 mm, vias 1 -> 0
- net Net-(J1-Pad5): track 36.5 -> 0.00 mm, vias 1 -> 0
- net Net-(J1-Pad3): track 34.3 -> 0.00 mm, vias 1 -> 0
- net PSI: track 21.2 -> 4.07 mm
- net PSD: track 26.7 -> 11.0 mm
- net PSO: track 20.8 -> 6.42 mm
- net PSC: track 17.9 -> 3.73 mm
- net GND: track 0.00 -> 6.46 mm
- removed copper zone on B.Cu, net GND
Other:
- board size 52.8 x 32.5 mm -> 14.2 x 32.5 mm
- board text added: "3v3"
- board text added: "GND 28"
- board text added: "PSC"
- board text added: "PSD"
- board text added: "PSI"
- board text added: "PSO"
- board text added: "Pico goes here lol"
- board text added: "Solder port on other side"
- board text added: "TileWorld GBA Thingamabob Made by: Matthew Collier (Squaresweets) Thanks to: DFranx, Nonchip, Lorenzoone, EchelonPrime, Stacksmashing and maciel310 for making this project possible!"
- board text removed: "5v"
- board text removed: "Little bit of extra space for wiring"
- board text removed: "Oh no! Your Raspberry pi Pico has been stolen! (Totally didn't steal that joke from Stacksmashing)"
- board text removed: "TileWorld adapter v.1 Made by: Matthew Collier (Squaresweets) Thanks to: DFranx, Nonchip, Lorenzoone, EchelonPrime, Stacksmashing and maciel310 for making this project possible!"
- board text removed: "level shifter thingamabobs"
