File: Hardware/Adapter/Adapter.kicad_sch (KiCad schematic)
At the start: 14 parts, among them J1 GameBoy_LinkPort, Q1 BSS13B, Q2 BSS13B, Q3 BSS13B, Q4 BSS13B, U1 Pico

Commit message: try stuff lol
The official name of the adapter is now the TileWorld GBA thingamabob, don't @ me
Parts:
- removed Q1, Q2, Q3, Q4: BSS13B, Package_TO_SOT_SMD:SOT-23, symbol Device:Q_NMOS_GSD
- removed R1, R2, R3, R4, R5, R6, R7, R8: 10k, Resistor_SMD:R_0402_1005Metric, symbol Device:R
Connections:
- net PSC: now also J1.5 (SC), U1.27 (GPIO21); no longer U1.1 (GPIO0)
- net PSD: now also J1.4 (SD), U1.24 (GPIO18); no longer U1.5 (GPIO3)
- net PSI: now also J1.3 (SI), U1.26 (GPIO20); no longer U1.2 (GPIO1)
- net PSO: now also J1.2 (SO), U1.25 (GPIO19); no longer U1.4 (GPIO2)
- no-connect marks 30 -> 34
Other:
- note removed: "GPI00"
- note removed: "GPI01"
- note removed: "GPI02"
- note removed: "GPI03"
- note removed: "Level shifters"
- note removed: "Link Cable Connector"
- moved on the sheet: J1

Commit message: Redid adapter, almost done, but I just wanna code stuff now
Connections:
- net GND: no longer U1.13 (GND), U1.18 (GND), U1.23 (GND), U1.3 (GND), U1.33 (AGND), U1.38 (GND), U1.8 (GND)
- removed net +3V3: U1.36 (3V3)
- net +5V: no longer names the net of J1.1 (VDD)
- net +5V: no longer U1.40 (VBUS)
- no-connect marks 34 -> 1
